File: Project 2 keyboard/prototype 2/Prototype 2.kicad_sch (KiCad schematic)
At the start: 1 part

Commit message: Auto stash before rebase of "refs/heads/main"
Parts:
- added D2, D3, D4: 1N4148, Diode_THT:D_DO-35_SOD27_P7.62mm_Horizontal, symbol Diode:1N4148
